File: MCU Datalogger.kicad_pcb (KiCad board)
At the start: 2 copper layers, 48.1 x 33.1 mm, 30 parts, among them J1 Conn_01x04_Pin, J2 Conn_01x04_Pin, J3 Conn_01x09_Pin, J4 Conn_02x03_Odd_Even, U1 24LC1025, U2 DS1337S_, U3 24LC1025, U4 ATMEGA328P-AU, Y1 32.768 KHZ, Y2 16 MHZ

Commit message: updated 2layer pcb
Connections:
- J2 pad 4: /SCK -> /SCL
- R4 pad 2: /SCK -> /SCL
- U1 pad 6: /SCK -> /SCL
- U2 pad 6: /SCK -> /SCL
- U3 pad 6: /SCK -> /SCL
- U4 pad 28: /SCK -> /SCL
Routing:
- net /SCK: track 147.6 -> 20.5 mm, vias 7 -> 2
- net /SCL: track 0.00 -> 91.4 mm, vias 0 -> 8
